Commit message: Align MoveIt joint names with URDF

File: src/003_moveit_config/config/gazebo_robot_arm.urdf (robot description, URDF)
Before this commit: robot robot_arm, 7 links, 6 joints
Joints:
- removed joint Joint_1
- removed joint Joint_2
- removed joint Joint_3
- removed joint Joint_4
- removed joint Joint_5
- removed joint Joint_6
- added joint joint_1: type revolute, parent base_link, child Link_1, origin xyz=0 0 0.063 rpy=0 0 0, axis 0 0 -1, limit lower=-3.14 upper=3.14 effort=100 velocity=100
- added joint joint_2: type revolute, parent Link_1, child Link_2, origin xyz=0.044 0 0.0465 rpy=0 0 0, axis -1 0 0, limit lower=-3.14 upper=3.14 effort=100 velocity=100
- added joint joint_3: type revolute, parent Link_2, child Link_3, origin xyz=0 0 0.211 rpy=0 0 0, axis -1 0 0, limit lower=-3.14 upper=3.14 effort=100 velocity=100
- added joint joint_4: type revolute, parent Link_3, child Link_4, origin xyz=-0.0041003 0 0.1945 rpy=0 0 0, axis 1 0 0, limit lower=-3.14 upper=3.14 effort=100 velocity=100
- added joint joint_5: type revolute, parent Link_4, child Link_5, origin xyz=0.0396 0 0.0379 rpy=0 0 0, axis 0 0 1, limit lower=-3.14 upper=3.14 effort=100 velocity=100
- added joint joint_6: type revolute, parent Link_5, child Link_6, origin xyz=0.0379 0 0.0396 rpy=0 0 0, axis 1 0 0, limit lower=-3.14 upper=3.14 effort=100 velocity=100
